Commit message: config controller and comanipulation optimization untested

File: urdf/cardboard.urdf.xacro (robot description, xacro)
@@ -25,5 +25,5 @@
         <joint name="joint_1" type="revolute">
             <axis xyz="0 1 0"/>
-            <limit effort="1000.0" lower="0.0" upper="0.548" velocity="0.5"/>
+            <limit effort="1000.0" lower="-2.96705973" upper="2.96705973" velocity="0.5"/>
             <origin rpy="0 0 0" xyz="${length/(joints+1)} 0.0 0"/>
             <parent link="base_link"/>
@@ -42,5 +42,5 @@
         <joint name="joint_2" type="revolute">
             <axis xyz="0 1 0"/>
-            <limit effort="1000.0" lower="0.0" upper="0.548" velocity="0.5"/>
+            <limit effort="1000.0" lower="-2.96705973" upper="2.96705973" velocity="0.5"/>
             <origin rpy="0 0 0" xyz="${length/(joints+1)} 0.0 0"/>
             <parent link="link_1"/>
@@ -59,5 +59,5 @@
         <joint name="joint_3" type="revolute">
             <axis xyz="0 1 0"/>
-            <limit effort="1000.0" lower="0.0" upper="0.548" velocity="0.5"/>
+            <limit effort="1000.0" lower="-2.96705973" upper="2.96705973" velocity="0.5"/>
             <origin rpy="0 0 0" xyz="${length/(joints+1)} 0.0 0"/>
             <parent link="link_2"/>
@@ -76,5 +76,5 @@
         <joint name="joint_4" type="revolute">
             <axis xyz="0 1 0"/>
-            <limit effort="1000.0" lower="0.0" upper="0.548" velocity="0.5"/>
+            <limit effort="1000.0" lower="-2.96705973" upper="2.96705973" velocity="0.5"/>
             <origin rpy="0 0 0" xyz="${length/(joints+1)} 0.0 0"/>
             <parent link="link_3"/>
@@ -93,5 +93,5 @@
         <joint name="joint_5" type="revolute">
             <axis xyz="0 1 0"/>
-            <limit effort="1000.0" lower="0.0" upper="0.548" velocity="0.5"/>
+            <limit effort="1000.0" lower="-2.96705973" upper="2.96705973" velocity="0.5"/>
             <origin rpy="0 0 0" xyz="${length/(joints+1)} 0.0 0"/>
             <parent link="link_4"/>
