Commit message: corrected urdf robot name

File: urdf/baxter_box.urdf (robot description, URDF)
Before this commit: robot cardboard, 62 links, 61 joints
Joints:
- joint joint_baxter_box: origin xyz=0 0 0 rpy=0 0 0 -> xyz=0 0 0 rpy=0 -1.57079632679 1.57079632679; parent l_gripper_l_finger_tip -> l_gripper_l_finger

File: urdf/baxter_box.urdf.xacro (robot description, xacro)
@@ -1,4 +1,4 @@
 <?xml version="1.0"?>
-<robot xmlns:xacro="http://www.ros.org/wiki/xacro" name="cardboard">
+<robot xmlns:xacro="http://www.ros.org/wiki/xacro" name="baxter_box">
     <xacro:include filename="box_chain.urdf.xacro"/>
     <xacro:include filename="$(find baxter_description)/urdf/baxter.urdf.xacro" ns="baxter"/>
