Commit message: box sim working without gravity

File: urdf/box.urdf (robot description, URDF)
Before this commit: robot box, 5 links, 4 joints
Joints:
- joint joint_3: axis (none) -> 0 1 0; limit (none) -> lower=-3.14159265359 upper=3.14159265359 effort=1000.0 velocity=1.5; type fixed -> revolute

File: urdf/box_chain.urdf.xacro (robot description, xacro)
@@ -80,5 +80,7 @@
             <child link="flap_2"/>
         </joint>
-        <joint name="joint_3" type="fixed">
+        <joint name="joint_3" type="revolute">
+            <axis xyz="0 1 0"/>
+            <limit effort="1000.0" lower="${-deg180}" upper="${deg180}" velocity="1.5"/>
             <origin rpy="0 0 0" xyz="${flap_length} 0 0"/>
             <parent link="flap_2"/>
